File: PdSinkInspector.kicad_sch (KiCad schematic)
At the start: 3 parts, among them IC1 632723100011, IC2 STUSB4700YQTR, U1 RP2040

Commit message: [Update]RP2040を結線
Parts:
- added C1, C10, C2, C3, C4, C5, C6, C7, C9: 0.1u, Capacitor_SMD:C_0603_1608Metric, symbol Device:C
- added C11, C8: 1u, Capacitor_SMD:C_0603_1608Metric, symbol Device:C
- added H1, H2, H3, H4: MountingHole, MountingHole:MountingHole_3.2mm_M3, symbol Mechanical:MountingHole
- added R1, R2: 27, Resistor_SMD:R_0603_1608Metric, symbol Device:R
- IC2: footprint QFN50P400X400X90-25N-D -> TE-01:QFN50P400X400X90-25N-D
Connections:
- net GND: now also U1.19 (TESTEN), U1.57 (GND), C1.2, C10.2, C11.2, C2.2, C3.2, C4.2, C5.2, C6.2, C7.2, C8.2, C9.2
- net USB_D+: now reaches IC1.A6 (DP1)
- net USB_D+: now also IC1.B6 (DP2), R1.1
- net USB_D-: now reaches IC1.A7 (DN1)
- net USB_D-: now also IC1.B7 (DN2), R2.1
- net +3.3V: now reaches U1.1 (IOVDD), U1.10 (IOVDD), U1.22 (IOVDD), U1.33 (IOVDD), U1.42 (IOVDD), U1.49 (IOVDD)
- net +3.3V: now also U1.43 (ADC_AVDD), U1.44 (VREG_IN), U1.48 (USB_VDD), C1.1, C2.1, C3.1, C4.1, C5.1, C6.1, C7.1, C8.1
- net +1V1: now reaches U1.23 (DVDD), U1.50 (DVDD)
- net +1V1: now also U1.45 (VREG_VOUT), C10.1, C11.1, C9.1
- net at U1.46 (USB_DM): now also R2.2
- net at U1.47 (USB_DP): now also R1.2
- net I2C1_SDA: now reaches U1.8 (GPIO6)
- net I2C1_SDA: now also IC2.8 (SDA)
- net I2C1_SCL: now reaches U1.9 (GPIO7)
- net I2C1_SCL: now also IC2.7 (SCL)
- no-connect marks 0 -> 2
Other:
- note added: "ネジ穴"
- moved on the sheet: IC1, IC2, U1
