File: PdSinkInspector.kicad_sch (KiCad schematic)
At the start: 34 parts, among them IC1 632723100011, IC2 STUSB4700YQTR, IC3 632723100011, SW1 SW_Omron_B3FS, U1 RP2040, U2 W25Q128JVS, U3 TLV75733PDBV, Y1 ABMM2-12.000MHZ-E2-T

Commit message: 2025/03/30
Parts:
- removed IC1, IC3: 632723100011, TE-01:632723100011, symbol TE-01:632723100011
- removed U3: TLV75733PDBV, Package_TO_SOT_SMD:SOT-23-5, symbol Regulator_Linear:TLV75733PDBV
- added C17: 0.1u, Capacitor_SMD:C_0603_1608Metric, symbol Device:C
- added C18, C19: 10u, Capacitor_SMD:C_0603_1608Metric, symbol Device:C
- added C20, C21: 1u, Capacitor_SMD:C_0603_1608Metric, symbol Device:C
- added D1: LED, LED_SMD:LED_0603_1608Metric, symbol Device:LED
- added J1, J2: USB_C_Receptacle, Connector_USB:USB_C_Receptacle_Molex_105450-0101, symbol Connector:USB_C_Receptacle
- added L1: 1.5u, Inductor_SMD:L_0805_2012Metric, symbol Device:L
- added Q1, Q2, Q3: AO3401A, Package_TO_SOT_SMD:SOT-23, symbol Transistor_FET:AO3401A
- added R10: 2k2, Resistor_SMD:R_0603_1608Metric, symbol Device:R
- added R11, R12, R8, R9: 10k, Resistor_SMD:R_0603_1608Metric, symbol Device:R
- added R7: 1k, Resistor_SMD:R_0603_1608Metric, symbol Device:R
- added U3: TPS63031DSK, Package_SON:WSON-10-1EP_2.5x2.5mm_P0.5mm_EP1.2x2mm, symbol Regulator_Switching:TPS63031DSK
- C1, C10, C12, C14, C2, C3, C4, C5, C6, C7, C9: BOM (none) -> C14663
- C11, C8: BOM (none) -> C15849
- C13: value 0.1u -> 10u; BOM (none) -> C14663
- C15, C16: BOM (none) -> C107045
- IC2: BOM (none) -> C2156427
- R1, R2: BOM (none) -> C4177
- R4: value 27 -> 100k; BOM (none) -> C4177
- R6: BOM (none) -> C21190
- U1: BOM (none) -> C2040
- U2: BOM (none) -> C97521
- Y1: BOM (none) -> C6117540
Connections:
- net +3.3V: now also R8.1; no longer C14.1
- net BOOT: now also SW1.2, C17.1, R8.2
- net GND: now also IC2.3 (VCONN), IC2.6 (RESET), SW1.1, C17.2, C18.2, C19.2, C20.2, C21.2, D1.1 (K), J1.A1 (GND), J1.A12 (GND), J1.B1 (GND), J1.B12 (GND), J1.S1 (SHIELD), J2.A1 (GND), J2.A12 (GND), J2.B1 (GND), J2.B12 (GND), J2.S1 (SHIELD), R12.1, U3.11 (PGND), U3.3 (PGND), U3.9 (GND)
- net USB_D+: now also J1.A6 (D+), J1.B6 (D+)
- net USB_D-: now also J1.A7 (D-), J1.B7 (D-)
- net VBUS: now also IC2.22 (VSYS), IC2.24 (VDD), J1.A4 (VBUS), J1.A9 (VBUS), J1.B4 (VBUS), J1.B9 (VBUS), R7.1, U3.5 (VIN)
- net at IC2.2 (CC1): now also J2.A5 (CC1)
- net at IC2.4 (CC2): now also J2.B5 (CC2)
- net at R4.2: now also IC2.13 (VVAR_ADDR0)
- net Vout: now reaches IC2.18 (VBUS_SENSE)
- net Vout: now also J2.A4 (VBUS), J2.A9 (VBUS), J2.B4 (VBUS), J2.B9 (VBUS)
- net at IC2.19 (VBUS_DISCH): now also Q3.1 (G), R11.1
- net at IC2.20 (VBUS_EN_SRC): now also R10.1
- net at IC2.21 (VREG_1V2): now also C20.1
- net at IC2.23 (VREG_2V7): now also C21.1
- net X_IN: no longer names the net of C15.1, U1.20 (XIN), Y1.1 (X1)
- net X_OUT: no longer names the net of R6.1, U1.21 (XOUT)
- new net: Q2.3 (D), Q3.2 (S), R11.2
- new net: D1.2 (A), R7.2
- new net: Q1.1 (G), Q2.1 (G), R10.2, R9.1
- new net: Q1.2 (S), Q2.2 (S), R9.2
- new net: C18.1, C19.1, U3.1 (VOUT), U3.10 (FB)
- new net: Q3.3 (D), R12.2
- new net: L1.1, U3.4 (L1)
- new net: L1.2, U3.2 (L2)
- new net: C14.1, U3.6 (EN), U3.7 (PS/SYNC), U3.8 (VINA)
- no-connect marks 15 -> 36
Other:
- note added: "PWR_FLAG(お作法)"
- moved on the sheet: C1, C10, C11, C12, C15, C16, C2, C3, C4, C5, C6, C7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

Commit message: i2cにプルアップ追加+JLC用にBOM作成(途中)
Parts:
- removed SW1: SW_Omron_B3FS, Button_Switch_SMD:SW_SPST_Omron_B3FS-105xP, symbol Switch:SW_Omron_B3FS
- removed Y1: ABMM2-12.000MHZ-E2-T, TE-01:ABMM2, symbol TE-01:ABMM2-12.000MHZ-E2-T
- added D2: SS14, Diode_SMD:D_SMA, symbol Diode:SS14
- added R13: 5.1, Resistor_SMD:R_0603_1608Metric, symbol Device:R
- added R14: 5.1k, Resistor_SMD:R_0603_1608Metric, symbol Device:R
- added R15, R16: 4.7k, Resistor_SMD:R_0603_1608Metric, symbol Device:R
- added SW1, SW2: SW_MEC_5E, TE-01:ABMM2, symbol Switch:SW_MEC_5E
- added Y2: Crystal_GND24, Crystal:Crystal_SMD_3225-4Pin_3.2x2.5mm, symbol Device:Crystal_GND24
- R5: value NC -> 1k
- U3: BOM (none) -> C15516
Connections:
- net +3.3V: now also C18.1, C19.1, U3.1 (VOUT), U3.10 (FB), R15.1, R16.1
- net BOOT: now also SW2.1, SW2.2; no longer C17.1, R8.2
- net GND: now also IC2.25 (EP), R13.2, R14.2, SW1.3 (K), SW1.4 (A), SW2.3 (K), Y2.2, Y2.4
- net I2C1_SCL: now also R15.2
- net I2C1_SDA: now also R16.2
- net VBUS: now also Q2.3 (D), Q3.2 (S), R11.2, D2.1 (K); no longer J1.A4 (VBUS), J1.A9 (VBUS), J1.B4 (VBUS), J1.B9 (VBUS)
- net Vout: now also Q1.3 (D)
- net at C16.1: now also R6.1, Y2.1; no longer R6.2
- net at C15.1, U1.20 (XIN): now also Y2.3
- net at U1.21 (XOUT): now also R6.2; no longer R6.1
- net RESET: now reaches U1.26 (RUN)
- net RESET: now also C17.1, R8.2, SW1.1, SW1.2
- net at J1.A5 (CC1): now also R14.1
- net at J1.B5 (CC2): now also R13.1
- new net: D2.2 (A), J1.A4 (VBUS), J1.A9 (VBUS), J1.B4 (VBUS), J1.B9 (VBUS)
- no-connect marks 36 -> 35
Other:
- moved on the sheet: C13, C14, C15, C16, C17, C18, C19, D1, J1, L1, Q1, Q2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

Commit message: LCSCセット
Parts:
- added R17: NC, Resistor_SMD:R_0603_1608Metric, symbol Device:R
- L1: BOM (none) -> C2042639
- R11, R12, R9: BOM C4177 -> C25804
- R13: value 5.1 -> 5.1k; BOM C21190 -> C23186
- R14: BOM C21190 -> C23186
- R5: BOM (none) -> C21190
Connections:
- net at C15.1, U1.20 (XIN), Y2.3: now also R17.2
- net at R6.2, U1.21 (XOUT): now also R17.1
Other:
- moved on the sheet: C13, C14, C18, C19, D1, D2, J1, L1, R13, R14, R6, R7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

Commit message: [Update]基板配置してみた
Parts:
- added D3, D4, D5: D, Diode_SMD:D_SOD-882, symbol Device:D
- Q1, Q2, Q3: BOM (none) -> C15127
Connections:
- net GND: now also D3.2 (A), D4.2 (A), D5.2 (A)
- net USB_D+: now also D4.1 (K)
- net USB_D-: now also D5.1 (K)
- net at D2.2 (A), J1.A4 (VBUS), J1.A9 (VBUS)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: now also D3.1 (K)
Other:
- moved on the sheet: J1, R13, R14

Commit message: [Update]基板配線開始+チップを0402に変更
Parts:
- removed J1, J2: USB_C_Receptacle, Connector_USB:USB_C_Receptacle_Molex_105450-0101, symbol Connector:USB_C_Receptacle
- added J1, J3: USB_C_Receptacle_USB2.0_16P, Connector_USB:USB_C_Receptacle_G-Switch_GT-USB-7010ASV, symbol Connector:USB_C_Receptacle_USB2.0_16P
- C1, C10, C12, C14, C17, C2, C3, C4, C5, C6, C7, C9: footprint Capacitor_SMD:C_0603_1608Metric -> Capacitor_SMD:C_0402_1005Metric; BOM C14663 -> C1525
- C11, C20, C21, C8: footprint Capacitor_SMD:C_0603_1608Metric -> Capacitor_SMD:C_0402_1005Metric; BOM C15849 -> C52923
- C13, C18, C19: footprint Capacitor_SMD:C_0603_1608Metric -> Capacitor_SMD:C_0402_1005Metric; BOM C14663 -> C15525
- C15, C16: footprint Capacitor_SMD:C_0603_1608Metric -> Capacitor_SMD:C_0402_1005Metric; BOM C107045 -> C1557
- R1, R2: footprint Resistor_SMD:R_0603_1608Metric -> Resistor_SMD:R_0402_1005Metric; BOM C4177 -> C25100
- R10: footprint Resistor_SMD:R_0603_1608Metric -> Resistor_SMD:R_0402_1005Metric; BOM C4177 -> C25879
- R11, R12, R8, R9: footprint Resistor_SMD:R_0603_1608Metric -> Resistor_SMD:R_0402_1005Metric; BOM C25804 -> C25744
- R13, R14: footprint Resistor_SMD:R_0603_1608Metric -> Resistor_SMD:R_0402_1005Metric; BOM C23186 -> C25905
- R15, R16: footprint Resistor_SMD:R_0603_1608Metric -> Resistor_SMD:R_0402_1005Metric; BOM C21190 -> C25900
- R4: footprint Resistor_SMD:R_0603_1608Metric -> Resistor_SMD:R_0402_1005Metric; BOM C4177 -> C25741
- R5, R6, R7: footprint Resistor_SMD:R_0603_1608Metric -> Resistor_SMD:R_0402_1005Metric; BOM C21190 -> C11702
Connections:
- net GND: now also J1.A1 (GND), J1.A12 (GND), J1.B1 (GND), J1.B12 (GND), J1.S1 (SHIELD), J3.A1 (GND), J3.A12 (GND), J3.B1 (GND), J3.B12 (GND), J3.S1 (SHIELD)
- net USB_D+: now also J3.A6 (D+), J3.B6 (D+)
- net USB_D-: now also J3.A7 (D-), J3.B7 (D-)
- net Vout: now also J1.A4 (VBUS), J1.A9 (VBUS), J1.B4 (VBUS), J1.B9 (VBUS)
- net at R14.1: now also J3.A5 (CC1)
- net at D2.2 (A), D3.1 (K): now also J3.A4 (VBUS), J3.A9 (VBUS), J3.B4 (VBUS), J3.B9 (VBUS)
- net at R13.1: now also J3.B5 (CC2)
- net at IC2.2 (CC1): now also J1.A5 (CC1)
- net at IC2.4 (CC2): now also J1.B5 (CC2)
- no-connect marks 35 -> 19
