File: PdSinkInspector.kicad_sch (KiCad schematic)
At the start: 65 parts, among them IC2 STUSB4700YQTR, J1 USB_C_Receptacle_USB2.0_16P, J2 Conn_01x12_Socket, J3 USB_C_Receptacle_USB2.0_16P, Q1 AO3401A, Q2 AO3401A, Q3 AO3401A, SW1 SW_MEC_5E, SW2 SW_MEC_5E, U1 RP2040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

Commit message: [Update]ガーバー作成
Parts:
- C1, C10, C12, C14, C17, C2, C22, C23, C3, C4, C5, C6, C7, C9: value 0.1u -> 0.1uF
- C11, C20, C21, C8: value 1u -> 1uF
- C13, C18, C19: value 10u -> 10uF
- C15, C16: value 27p -> 27pF
- J1, J3: BOM (none) -> C2988369
- J2: BOM (none) -> C596811
- L1: value 1.5u -> 1.5uH
- R18: BOM (none) -> C25077
- U4: BOM (none) -> C891320
Connections:
- net GND: now also SW2.4 (A)
Changed lines of the file:
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@@
 	(paper "A4")
 	(junction
-		(at 186.69 68.58)
+		(at 179.07 68.58)
 		(diameter 0)
 		(color 0 0 0 0)
@@
 	)
 	(junction
-		(at 186.69 71.12)
+		(at 179.07 71.12)
 		(diameter 0)
 		(color 0 0 0 0)
@@
 	)
 	(junction
-		(at 186.69 66.04)
+		(at 179.07 66.04)
 		(diameter 0)
 		(color 0 0 0 0)
@@
 	)
 	(junction
+		(at 237.49 2.54)
+		(diameter 0)
+		(color 0 0 0 0)
+	)
+	(junction
 		(at 234.95 73.66)
 		(diameter 0)
@@
 	(wire
 		(pts
-			(xy 186.69 68.58) (xy 199.39 68.58)
+			(xy 179.07 68.58) (xy 199.39 68.58)
 		)
 		(stroke
@@
 	(wire
 		(pts
-			(xy 186.69 66.04) (xy 199.39 66.04)
+			(xy 179.07 66.04) (xy 199.39 66.04)
 		)
 		(stroke
@@
 	(wire
 		(pts
-			(xy 186.69 50.8) (xy 186.69 66.04)
+			(xy 179.07 50.8) (xy 179.07 66.04)
 		)
 		(stroke
@@
 	(wire
 		(pts
-			(xy 186.69 66.04) (xy 186.69 68.58)
+			(xy 179.07 66.04) (xy 179.07 68.58)
 		)
 		(stroke
@@
 	(wire
 		(pts
+			(xy 237.49 2.54) (xy 240.03 2.54)
+		)
+		(stroke
+			(width 0)
+			(type default)
+		)
+	)
+	(wire
+		(pts
 			(xy 425.45 -58.42) (xy 425.45 -62.23)
 		)
@@
 	(wire
 		(pts
-			(xy 199.39 50.8) (xy 186.69 50.8)
+			(xy 199.39 50.8) (xy 179.07 50.8)
 		)
 		(stroke
@@
 	(wire
 		(pts
-			(xy 199.39 71.12) (xy 186.69 71.12)
+			(xy 199.39 71.12) (xy 179.07 71.12)
 		)
 		(stroke
@@
 	(wire
 		(pts
-			(xy 186.69 68.58) (xy 186.69 71.12)
+			(xy 179.07 68.58) (xy 179.07 71.12)
 		)
 		(stroke
@@
 	(wire
 		(pts
-			(xy 186.69 71.12) (xy 186.69 80.01)
+			(xy 179.07 71.12) (xy 179.07 80.01)
 		)
 		(stroke
@@
 			)
 		)
-		(property "Value" "27p"
+		(property "Value" "27pF"
 			(at 327.406 5.08 0)
 			(effects
@@
 			)
 		)
+		(property "BOM" "C2988369"
+			(at 542.29 8.89 0)
+			(effects
+				(font
+					(size 1.27 1.27)
+				)
+				(hide yes)
+			)
+		)
 		(pin "A1"
 		)
@@
 			)
 		)
-		(property "Value" "0.1u"
+		(property "Value" "0.1uF"
 			(at 283.464 -63.5 0)
 			(effects
@@
 			)
 		)
-		(property "Value" "0.1u"
+		(property "Value" "0.1uF"
 			(at 197.104 38.1 0)
 			(effects
@@
 			)
 		)
-		(property "Value" "0.1u"
+		(property "Value" "0.1uF"
 			(at 393.446 -82.55 0)
 			(effects
@@
 			)
 		)
-		(property "Value" "0.1u"
+		(property "Value" "0.1uF"
 			(at 423.926 -82.55 0)
 			(effects
@@
 			)
 		)
-		(property "Value" "0.1u"
+		(property "Value" "0.1uF"
 			(at 266.954 -1.27 0)
 			(effects
@@
 			)
 		)
-		(property "Value" "0.1u"
+		(property "Value" "0.1uF"
 			(at 220.726 38.1 0)
 			(effects
@@
 			)
 		)
+		(property "BOM" "C891320"
+			(at 209.55 60.96 0)
+			(effects
+				(font
+					(size 1.27 1.27)
+				)
+				(hide yes)
+			)
+		)
 		(pin "7"
 		)
@@
 			)
 		)
-		(property "Value" "10u"
+		(property "Value" "10uF"
 			(at 233.934 -50.8 0)
 			(effects
@@
 			)
 		)
-		(property "Value" "0.1u"
+		(property "Value" "0.1uF"
 			(at 416.306 -82.55 0)
 			(effects
@@
 			)
 		)
-		(property "Value" "0.1u"
+		(property "Value" "0.1uF"
 			(at 401.066 -82.55 0)
 			(effects
@@
 			)
 		)
-		(property "Value" "0.1u"
+		(property "Value" "0.1uF"
 			(at 439.166 -82.55 0)
 			(effects
@@
 			)
 		)
-		(property "Value" "27p"
+		(property "Value" "27pF"
 			(at 310.134 5.08 0)
 			(effects
@@
 			)
 		)
-		(property "Value" "0.1u"
+		(property "Value" "0.1uF"
 			(at 356.616 -82.55 0)
 			(effects
@@
 			)
 		)
-		(property "Value" "10u"
+		(property "Value" "10uF"
 			(at 242.824 -50.8 0)
 			(effects
@@
 			)
 		)
-		(property "Value" "1.5u"
+		(property "Value" "1.5uH"
 			(at 202.184 -41.91 0)
 			(effects
@@
 	(symbol
 		(lib_id "power:GND")
-		(at 186.69 80.01 0)
+		(at 179.07 80.01 0)
 		(unit 1)
 		(exclude_from_sim no)
@@
 		(fields_autoplaced yes)
 		(property "Reference" "#PWR051"
-			(at 186.69 86.36 0)
+			(at 179.07 86.36 0)
 			(effects
 				(font
@@
 		)
 		(property "Value" "GND"
-			(at 186.69 85.09 0)
+			(at 179.07 85.09 0)
 			(effects
 				(font
@@
 		)
 		(property "Footprint" ""
-			(at 186.69 80.01 0)
+			(at 179.07 80.01 0)
 			(effects
 				(font
@@
 		)
 		(property "Datasheet" ""
-			(at 186.69 80.01 0)
+			(at 179.07 80.01 0)
 			(effects
 				(font
@@
 		)
 		(property "Description" "Power symbol creates a global label with name \"GND\" , ground"
-			(at 186.69 80.01 0)
+			(at 179.07 80.01 0)
 			(effects
 				(font
@@
 			)
 		)
-		(property "Value" "0.1u"
+		(property "Value" "0.1uF"
 			(at 364.236 -82.55 0)
 			(effects
@@
 			)
 		)
-		(property "Value" "0.1u"
+		(property "Value" "0.1uF"
 			(at 194.564 -50.8 0)
 			(effects
@@
 			)
 		)
+		(property "BOM" "C25077"
+			(at 229.87 71.12 0)
+			(effects
+				(font
+					(size 1.27 1.27)
+				)
+				(hide yes)
+			)
+		)
 		(pin "2"
 		)
@@
 			)
 		)
-		(property "Value" "1u"
+		(property "Value" "1uF"
 			(at 448.056 -82.55 0)
 			(effects
@@
 			)
 		)
-		(property "Value" "10u"
+		(property "Value" "10uF"
 			(at 183.134 -50.8 0)
 			(effects
@@
 			)
 		)
-		(property "Value" "0.1u"
+		(property "Value" "0.1uF"
 			(at 431.546 -82.55 0)
 			(effects
@@
 			)
 		)
-		(property "Value" "1u"
+		(property "Value" "1uF"
 			(at 512.826 -34.29 0)
 			(effects
@@
 			)
 		)
+		(property "BOM" "C596811"
+			(at 243.84 63.5 0)
+			(effects
+				(font
+					(size 1.27 1.27)
+				)
+				(hide yes)
+			)
+		)
 		(pin "5"
 		)
@@
 			)
 		)
-		(property "Value" "1u"
+		(property "Value" "1uF"
 			(at 347.726 -82.55 0)
 			(effects
@@
 			)
 		)
-		(property "Value" "0.1u"
+		(property "Value" "0.1uF"
 			(at 408.686 -82.55 0)
 			(effects
@@
 			)
 		)
-		(property "Value" "1u"
+		(property "Value" "1uF"
 			(at 522.986 -34.29 0)
 			(effects
@@
 			(at 96.52 -43.18 0)
 			(effects
+				(font
+					(size 1.27 1.27)
+				)
+				(hide yes)
+			)
+		)
+		(property "BOM" "C2988369"
+			(at 96.52 -43.18 0)
+			(effects

Commit message: [Fix]不要なレベル変換を削除
Parts:
- removed C22, C23: 0.1uF, Capacitor_SMD:C_0402_1005Metric, symbol Device:C
- removed U4: FXMA108, Package_DFN_QFN:WQFN-20-1EP_2.5x4.5mm_P0.5mm_EP1x2.9mm, symbol Logic_LevelTranslator:FXMA108
Connections:
- net Data/Command: now also J2.7 (Pin_7)
- net LCD_RESET: now also J2.11 (Pin_11)
- net MOSI: now also J2.10 (Pin_10)
- net SPI_CS: now also J2.8 (Pin_8)
- net SPI_SCK: now also J2.9 (Pin_9)
Other:
- note added: "MCU&PD_IC"
- note added: "SW"
- note added: "USB Input"
- moved on the sheet: C1, C10, C11, C12, C13, C14, C15, C16, C17, C18, C19, C2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
