File: _autosave-PdSinkInspector.kicad_sch (KiCad schematic)
At the start: 65 parts, among them IC2 STUSB4700YQTR, J1 USB_C_Receptacle_USB2.0_16P, J2 Conn_01x12_Socket, J3 USB_C_Receptacle_USB2.0_16P, Q1 AO3401A, Q2 AO3401A, Q3 AO3401A, SW1 SW_MEC_5E, SW2 SW_MEC_5E, U1 RP2040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

Commit message: 4/13進捗
Changed lines of the file:
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@@
 		(at 443.23 -21.59)
+	)
+	(bus_entry
+		(at 203.2 77.47)
+		(size 2.54 2.54)
+		(stroke
+			(width 0)
+			(type default)
+		)
 	)
 	(wire
